Commit message: feat(fase7): fecha Fase 7 com AP_DDS auto-start, mixer Lua V5 e missao WP1->WP2
Consolida o trabalho da Fase 7 (ArduPilot SITL + Gazebo Harmonic + AP_DDS + QGroundControl) e adiciona o fix de race condition no auto-start do micro-ros-agent identificado em 2026-05-06.

Mudancas principais:

- sim.launch.py: integra ArduPilot SITL (sim_vehicle.py Rover JSON), micro-ros-agent (udp4:2019) e mavlink_bridge_node sob a flag ardupilot:=true. Adiciona respawn=True/respawn_delay=2.0 no agent e reordena timings (agent t=10s, SITL t=18s, bridge t=28s) para resolver "DDS: No ping response, exiting" causado pelo SITL pingar o agent antes do bind UDP.
- asv_mavlink/mavlink_bridge_node.py: bridge MAVLink que le SERVO_OUTPUT_RAW e publica /model/migbot/joint/Engine_helice_N/cmd_vel para o gz-sim-thruster-system gerar empuxo fisico.
- asv_mavlink/fase7_sanity_check.py: teste automatizado SERVO_OUTPUT_RAW -> cmd_vel -> force -> pose.
- migbot.urdf.xacro: ArduPilotPlugin configurado, controles dos 6 canais em VELOCITY, gazeboXYZToNED ajustado, spawn invertido (-R 3.14159).
- config/migbot_mixer.lua: Lua mixer V5 hibrido AP/RC (FRAME_CLASS=15, SERVO1..6_FUNCTION=94..99).
- config/migbot_sitl.param: parametros Rover SITL com DDS_ENABLE/DDS_UDP_PORT e tuning inicial de AUTO.
- madeira_river_simple.sdf: ajustes do mundo de teste.
- docs/FASE7_STATUS.md (novo): status operacional detalhado por subfase.
- docs/MOTOR_MIXER_DOSSIER.md (novo): dossie do problema de propulsao e licoes aprendidas.
- docs/FASE7_AP_DDS.md, docs/GUIA_FASES.md, docs/ARCHITECTURE.md, docs/SPAWN_TROUBLESHOOTING.md: atualizacoes refletindo Fase 7 fechada, fix de race AP_DDS, validacao WP1->WP2 em AUTO e limitacao conhecida (sem obstacle avoidance, escopo Fase 8).

Validacao 2026-05-06:
- Migbot navega em MANUAL e em AUTO via QGroundControl.
- /ap/pose/filtered ~20-25 Hz, /ap/twist/filtered ~22 Hz, /ap/navsat ~4.5 Hz.
- Transicao WP1 -> WP2 confirmada sem warning DDS.
- Limitacao: colisao em obstaculos do madeira_river_simple (a tratar na Fase 8).

File: src/asv_description/urdf/migbot.urdf.xacro (robot description, xacro)
@@ -128,5 +128,6 @@
     </collision>
     <inertial>
-      <origin xyz="0.387 0.095 0.15" rpy="0 0 0" />
+      <!-- CoM centralizado entre pontoes (Y=0.096) e abaixado (Z=0.05) para estabilidade lateral -->
+      <origin xyz="0.150 0.096 0.05" rpy="0 0 0" />
       <mass value="142.500037" />
       <inertia ixx="37.182755" ixy="0.0" ixz="0.0" iyy="70.128464" iyz="0.0" izz="92.883435" />
@@ -140,5 +141,5 @@
     <child link="Helice_1" />
     <origin xyz="1.0098435878753662 -0.5541407465934753 0.6604171991348267" rpy="0.0 0.0 0.0" />
-    <axis xyz="0 1 0" />
+    <axis xyz="1 0 0" />
     <dynamics damping="0.05" friction="0.05" />
   </joint>
@@ -147,5 +148,5 @@
     <child link="Helice_2" />
     <origin xyz="-0.34517043828964233 0.746247410774231 0.6604171991348267" rpy="0.0 0.0 0.0" />
-    <axis xyz="0 1 0" />
+    <axis xyz="1 0 0" />
     <dynamics damping="0.05" friction="0.05" />
   </joint>
@@ -154,5 +155,5 @@
     <child link="Helice_3" />
     <origin xyz="1.009843349456787 0.7462476491928101 0.6604171991348267" rpy="0.0 0.0 0.0" />
-    <axis xyz="0 1 0" />
+    <axis xyz="1 0 0" />
     <dynamics damping="0.05" friction="0.05" />
   </joint>
@@ -161,5 +162,5 @@
     <child link="Helice_4" />
     <origin xyz="-0.345170259475708 -0.5537497997283936 0.6604171991348267" rpy="0.0 0.0 0.0" />
-    <axis xyz="0 1 0" />
+    <axis xyz="1 0 0" />
     <dynamics damping="0.05" friction="0.05" />
   </joint>
@@ -168,5 +169,5 @@
     <child link="Helice_5" />
     <origin xyz="-0.7168807983398438 0.746498703956604 0.6604171991348267" rpy="0.0 0.0 0.0" />
-    <axis xyz="0 1 0" />
+    <axis xyz="1 0 0" />
     <dynamics damping="0.05" friction="0.05" />
   </joint>
@@ -175,5 +176,5 @@
     <child link="Helice_6" />
     <origin xyz="-0.7168805599212646 -0.5537497997283936 0.6604171991348267" rpy="0.0 0.0 0.0" />
-    <axis xyz="0 1 0" />
+    <axis xyz="1 0 0" />
     <dynamics damping="0.05" friction="0.05" />
   </joint>
@@ -228,10 +229,8 @@
   <!-- Sensores Gazebo (referências de link)                  -->
   <!-- ====================================================== -->
-  <gazebo reference="imu_link">
+  <gazebo reference="base_link">
     <sensor name="imu_sensor" type="imu">
       <always_on>1</always_on>
       <update_rate>50</update_rate>
-      <topic>imu</topic>
-      <gz_frame_id>imu_link</gz_frame_id>
       <imu>
         <angular_velocity><x><noise type="gaussian"><mean>0</mean><stddev>0.009</stddev></noise></x><y><noise type="gaussian"><mean>0</mean><stddev>0.009</stddev></noise></y><z><noise type="gaussian"><mean>0</mean><stddev>0.009</stddev></noise></z></angular_velocity>
@@ -240,16 +239,14 @@
     </sensor>
   </gazebo>
-  <gazebo reference="gps_link">
+  <gazebo reference="base_link">
     <sensor name="navsat_sensor" type="navsat">
       <always_on>1</always_on>
       <update_rate>5</update_rate>
-      <topic>navsat</topic>
     </sensor>
   </gazebo>
-  <gazebo reference="mag_link">
+  <gazebo reference="base_link">
     <sensor name="magnetometer_sensor" type="magnetometer">
       <always_on>1</always_on>
       <update_rate>20</update_rate>
-      <topic>magnetometer</topic>
     </sensor>
   </gazebo>
@@ -262,48 +259,48 @@
       <namespace>migbot</namespace>
       <joint_name>Engine_helice_1</joint_name>
-      <thrust_coefficient>0.004422</thrust_coefficient>
-      <fluid_density>997.8</fluid_density>
-      <propeller_diameter>0.08</propeller_diameter>
-      <use_angvel_cmd>false</use_angvel_cmd>
+      <thrust_coefficient>0.05</thrust_coefficient>
+      <fluid_density>997.8</fluid_density>
+      <propeller_diameter>0.2</propeller_diameter>
+      <use_angvel_cmd>true</use_angvel_cmd>
     </plugin>
     <plugin filename="gz-sim-thruster-system" name="gz::sim::systems::Thruster">
       <namespace>migbot</namespace>
       <joint_name>Engine_helice_2</joint_name>
-      <thrust_coefficient>0.004422</thrust_coefficient>
-      <fluid_density>997.8</fluid_density>
-      <propeller_diameter>0.08</propeller_diameter>
-      <use_angvel_cmd>false</use_angvel_cmd>
+      <thrust_coefficient>0.05</thrust_coefficient>
+      <fluid_density>997.8</fluid_density>
+      <propeller_diameter>0.2</propeller_diameter>
+      <use_angvel_cmd>true</use_angvel_cmd>
     </plugin>
     <plugin filename="gz-sim-thruster-system" name="gz::sim::systems::Thruster">
       <namespace>migbot</namespace>
       <joint_name>Engine_helice_3</joint_name>
-      <thrust_coefficient>0.004422</thrust_coefficient>
-      <fluid_density>997.8</fluid_density>
-      <propeller_diameter>0.08</propeller_diameter>
-      <use_angvel_cmd>false</use_angvel_cmd>
+      <thrust_coefficient>0.05</thrust_coefficient>
+      <fluid_density>997.8</fluid_density>
+      <propeller_diameter>0.2</propeller_diameter>
+      <use_angvel_cmd>true</use_angvel_cmd>
     </plugin>
     <plugin filename="gz-sim-thruster-system" name="gz::sim::systems::Thruster">
       <namespace>migbot</namespace>
       <joint_name>Engine_helice_4</joint_name>
-      <thrust_coefficient>0.004422</thrust_coefficient>
-      <fluid_density>997.8</fluid_density>
-      <propeller_diameter>0.08</propeller_diameter>
-      <use_angvel_cmd>false</use_angvel_cmd>
+      <thrust_coefficient>0.05</thrust_coefficient>
+      <fluid_density>997.8</fluid_density>
+      <propeller_diameter>0.2</propeller_diameter>
+      <use_angvel_cmd>true</use_angvel_cmd>
     </plugin>
     <plugin filename="gz-sim-thruster-system" name="gz::sim::systems::Thruster">
       <namespace>migbot</namespace>
       <joint_name>Engine_helice_5</joint_name>
-      <thrust_coefficient>0.004422</thrust_coefficient>
-      <fluid_density>997.8</fluid_density>
-      <propeller_diameter>0.08</propeller_diameter>
-      <use_angvel_cmd>false</use_angvel_cmd>
+      <thrust_coefficient>0.05</thrust_coefficient>
+      <fluid_density>997.8</fluid_density>
+      <propeller_diameter>0.2</propeller_diameter>
+      <use_angvel_cmd>true</use_angvel_cmd>
     </plugin>
     <plugin filename="gz-sim-thruster-system" name="gz::sim::systems::Thruster">
       <namespace>migbot</namespace>
       <joint_name>Engine_helice_6</joint_name>
-      <thrust_coefficient>0.004422</thrust_coefficient>
-      <fluid_density>997.8</fluid_density>
-      <propeller_diameter>0.08</propeller_diameter>
-      <use_angvel_cmd>false</use_angvel_cmd>
+      <thrust_coefficient>0.05</thrust_coefficient>
+      <fluid_density>997.8</fluid_density>
+      <propeller_diameter>0.2</propeller_diameter>
+      <use_angvel_cmd>true</use_angvel_cmd>
     </plugin>
     <!-- ========== HIDRODINÂMICA (SNAME) ========== -->
@@ -329,3 +326,116 @@
     </plugin>
   </gazebo>
+  <!-- ====================================================== -->
+  <!-- ArduPilot SITL Plugin (Fase 7B)                        -->
+  <!-- Formato seguindo iris_with_ardupilot/model.sdf oficial. -->
+  <!-- ====================================================== -->
+  <gazebo>
+    <plugin name="ArduPilotPlugin" filename="ArduPilotPlugin">
+      <fdm_addr>127.0.0.1</fdm_addr>
+      <fdm_port_in>9002</fdm_port_in>
+      <connectionTimeoutMaxCount>5</connectionTimeoutMaxCount>
+      <lock_step>1</lock_step>
+      <no_time_sync>1</no_time_sync>
+      <have_32_channels>0</have_32_channels>
+      <modelXYZToAirplaneXForwardZDown degrees="true">0 0 0 0 0 0</modelXYZToAirplaneXForwardZDown>
+      <gazeboXYZToNED degrees="true">0 0 0 180 0 90</gazeboXYZToNED>
+      <imuName>base_link::imu_sensor</imuName>
+      <control channel="0">
+        <jointName>Engine_helice_1</jointName>
+        <useForce>1</useForce>
+        <multiplier>100.0</multiplier>
+        <offset>-0.5</offset>
+        <servo_min>1000</servo_min>
+        <servo_max>2000</servo_max>
+        <type>VELOCITY</type>
+        <p_gain>1.0</p_gain>
+        <i_gain>0</i_gain>
+        <d_gain>0</d_gain>
+        <i_max>0</i_max>
+        <i_min>0</i_min>
+        <cmd_max>50.0</cmd_max>
+        <cmd_min>-50.0</cmd_min>
+      </control>
+      <control channel="1">
+        <jointName>Engine_helice_2</jointName>
+        <useForce>1</useForce>
+        <multiplier>100.0</multiplier>
+        <offset>-0.5</offset>
+        <servo_min>1000</servo_min>
+        <servo_max>2000</servo_max>
+        <type>VELOCITY</type>
+        <p_gain>1.0</p_gain>
+        <i_gain>0</i_gain>
+        <d_gain>0</d_gain>
+        <i_max>0</i_max>
+        <i_min>0</i_min>
+        <cmd_max>50.0</cmd_max>
+        <cmd_min>-50.0</cmd_min>
+      </control>
+      <control channel="2">
+        <jointName>Engine_helice_3</jointName>
+        <useForce>1</useForce>
+        <multiplier>100.0</multiplier>
+        <offset>-0.5</offset>
+        <servo_min>1000</servo_min>
+        <servo_max>2000</servo_max>
+        <type>VELOCITY</type>
+        <p_gain>1.0</p_gain>
+        <i_gain>0</i_gain>
+        <d_gain>0</d_gain>
+        <i_max>0</i_max>
+        <i_min>0</i_min>
+        <cmd_max>50.0</cmd_max>
+        <cmd_min>-50.0</cmd_min>
+      </control>
+      <control channel="3">
+        <jointName>Engine_helice_4</jointName>
+        <useForce>1</useForce>
+        <multiplier>100.0</multiplier>
+        <offset>-0.5</offset>
+        <servo_min>1000</servo_min>
+        <servo_max>2000</servo_max>
+        <type>VELOCITY</type>
+        <p_gain>1.0</p_gain>
+        <i_gain>0</i_gain>
+        <d_gain>0</d_gain>
+        <i_max>0</i_max>
+        <i_min>0</i_min>
+        <cmd_max>50.0</cmd_max>
+        <cmd_min>-50.0</cmd_min>
+      </control>
+      <control channel="4">
+        <jointName>Engine_helice_5</jointName>
+        <useForce>1</useForce>
+        <multiplier>100.0</multiplier>
+        <offset>-0.5</offset>
+        <servo_min>1000</servo_min>
+        <servo_max>2000</servo_max>
+        <type>VELOCITY</type>
+        <p_gain>1.0</p_gain>
+        <i_gain>0</i_gain>
+        <d_gain>0</d_gain>
+        <i_max>0</i_max>
+        <i_min>0</i_min>
+        <cmd_max>50.0</cmd_max>
+        <cmd_min>-50.0</cmd_min>
+      </control>
+      <control channel="5">
+        <jointName>Engine_helice_6</jointName>
+        <useForce>1</useForce>
+        <multiplier>100.0</multiplier>
+        <offset>-0.5</offset>
+        <servo_min>1000</servo_min>
+        <servo_max>2000</servo_max>
+        <type>VELOCITY</type>
+        <p_gain>1.0</p_gain>
+        <i_gain>0</i_gain>
+        <d_gain>0</d_gain>
+        <i_max>0</i_max>
+        <i_min>0</i_min>
+        <cmd_max>50.0</cmd_max>
+        <cmd_min>-50.0</cmd_min>
+      </control>
+    </plugin>
+  </gazebo>
 </robot>
